Commit message: update for torque control on ROS1

File: dsr_description/xacro/m0609.urdf.xacro (robot description, xacro)
@@ -3,8 +3,15 @@
   <xacro:arg name="color"   default="white"/>
   <xacro:arg name="gripper" default="none"/>
+  <xacro:arg name="controller" default="position"/>
   <xacro:property name="cr" value="$(arg color)"/>
   <xacro:property name="gr" value="$(arg gripper)"/>
+  <xacro:property name="ctrl" value="$(arg controller)"/>
   <xacro:if value="${cr == 'white'}">
+    <xacro:if value="${ctrl == 'position'}">
      <xacro:include filename="$(find dsr_description)/xacro/macro.m0609.white.xacro" />
+    </xacro:if>
+    <xacro:if value="${ctrl == 'torque'}">
+     <xacro:include filename="$(find dsr_description)/xacro/macro.m0609.white.torque.xacro" />
+    </xacro:if>
   </xacro:if>
   <xacro:if value="${cr == 'blue'}">
