Commit message: update

File: dsr_description/urdf/m0609.urdf (robot description, URDF)
Before this commit: robot m0609, 8 links, 7 joints
Links:
- link base_0: mass 3.722 -> 3.18
- link link1: mass 7.446 -> 5.02
- link link2: mass 10.569 -> 8.04
- link link3: mass 3.614 -> 3.6
- link link4: mass 3.785 -> 3.57
- link link5: mass 2.598 -> 2.83
- link link6: mass 1.128 -> 1.16
Joints:
- joint joint1: origin xyz=0 0 0.1525 rpy=0 0 0 -> xyz=0 0 0.135 rpy=0 0 0
- joint joint2: origin xyz=0 0.006 0 rpy=0 -1.571 -1.571 -> xyz=0 0.0062 0 rpy=0 -1.571 -1.571

File: dsr_description/xacro/macro.m0609.white.xacro (robot description, xacro)
@@ -25,5 +25,5 @@
 			<parent link="base_0" />
 			<child link="link1" />
-			<origin rpy="0 0 0" xyz="0 0 0.1" />
+			<origin rpy="0 0 0" xyz="0 0 0.135" />
 			<axis xyz="0 0 1" />
 			<limit effort="163" lower="-6.2832" upper="6.2832" velocity="2.618"/>
